Commit message: jsp gui and inertial urdf

File: src/my_robot_description/urdf/robot_core.xacro (robot description, xacro)
@@ -1,4 +1,5 @@
 <?xml version="1.0"?>
 <robot xmlns:xacro="http://www.ros.org/wiki/xacro">
+    <xacro:include filename="inertial_macros.xacro"/>
     <material name="white">
         <color rgba="1 1 1 1" />
@@ -36,4 +37,7 @@
             </geometry>
         </collision>
+        <xacro:inertial_box mass="0.5" x="0.3" y="0.3" z="0.15">
+            <origin xyz="0.15 0 0.075" rpy="0 0 0"/>
+        </xacro:inertial_box>
     </link>
     <!-- LEFT WHEEL LINK -->
@@ -41,5 +45,5 @@
         <parent link="base_link"/>
         <child link="left_wheel"/>
-        <origin xyz="0 0.175 0" rpy="-${pi/2} 0 0"/>
+        <origin xyz="0 0.175 0" rpy="-1.57079632679 0 0"/>
         <axis xyz="0 0 1"/>
     </joint>
@@ -56,4 +60,7 @@
             </geometry>
         </collision>
+        <xacro:inertial_cylinder mass="0.1" length="0.04" radius="0.05">
+            <origin xyz="0 0 0" rpy="0 0 0"/>
+        </xacro:inertial_cylinder>
     </link>
     <!-- RIGHT WHEEL LINK -->
@@ -61,5 +68,5 @@
         <parent link="base_link"/>
         <child link="right_wheel"/>
-        <origin xyz="0 -0.175 0" rpy="${pi/2} 0 0"/>
+        <origin xyz="0 -0.175 0" rpy="1.57079632679 0 0"/>
         <axis xyz="0 0 -1"/>
     </joint>
@@ -76,4 +83,7 @@
             </geometry>
         </collision>
+        <xacro:inertial_cylinder mass="0.1" length="0.04" radius="0.05">
+            <origin xyz="0 0 0" rpy="0 0 0"/>
+        </xacro:inertial_cylinder>
     </link>
     <!-- CASTER WHEEL LINK -->
@@ -95,4 +105,7 @@
             </geometry>
         </collision>
+        <xacro:inertial_sphere mass="0.1" radius="0.05">
+            <origin xyz="0 0 0" rpy="0 0 0"></origin>
+        </xacro:inertial_sphere>
     </link>
 </robot>
